Commit message: Updated simulation with working first segment

File: simulation/arm.urdf (robot description, URDF)
Before this commit: robot arm, 10 links, 9 joints
Links:
- link base_link: mass 1.0 -> 0.001
- link hand: mass 0.5 -> 0.001
- link motor0: mass 0.5 -> 0.001
- link motor1: mass 0.5 -> 0.001
- link motor2: mass 0.5 -> 0.001
- link motor3: mass 0.5 -> 0.001
- link motor4: mass 0.5 -> 0.001
- link motor5: mass 0.5 -> 0.001
- link segment1: mass 1 -> 0.001
- link segment2: mass 1 -> 0.001
Joints:
- joint joint1: limit effort=10 velocity=3 -> effort=5000 velocity=1000
- joint joint2: limit effort=10 velocity=3 -> effort=1000 velocity=3000
- joint joint3: limit effort=10 velocity=3 -> effort=1000 velocity=3000
- joint joint5: limit effort=10 velocity=3 -> effort=1000 velocity=3000
- joint joint6: limit effort=10 velocity=3 -> effort=1000 velocity=3000
- joint joint8: limit effort=10 velocity=3 -> effort=1000 velocity=3000
